Commit message: Change the position of the laser and reset the angle info

File: robo_shield_pkg/urdf/hokuyo_right.xacro (robot description, xacro)
@@ -22,5 +22,5 @@
       <origin xyz="0 0 0" rpy="1.57 0 1.57"/>
       <geometry>
-        <mesh filename="/home/huang_uyhsp/catkin_ws/src/robo_shield_pkg/meshes/hokuyo.dae"/>
+        <mesh filename="$(find robo_shield_pkg)/meshes/hokuyo.dae"/>
       </geometry>
     </visual>
